File: hardware/inputsheild_4.brd (EAGLE design)
At the start: 71.1 x 90 mm, 89 parts

Commit message: hardware
Parts:
- renumbered TRG to TRIG, TRG_ to TRIG_
Connections:
- new net SLR: B1.D5
- net SFR: no longer B1.D5
Routing:
- net SFR: track 0.00 -> 214.2 mm, vias 0 -> 5
- net ER: track 0.00 -> 185.9 mm, vias 0 -> 6
- net TRIG: track 0.00 -> 174.6 mm, vias 0 -> 2
- net SRF: track 0.00 -> 164.9 mm, vias 0 -> 4
- net SRB: track 0.00 -> 160.5 mm, vias 0 -> 9
- net EF: track 0.00 -> 157.7 mm, vias 0 -> 6
- net SBL: track 0.00 -> 156.5 mm, vias 0 -> 6
- net EL: track 0.00 -> 156.3 mm, vias 0 -> 5
- net +5V: track 0.00 -> 153.7 mm, vias 0 -> 3
- net EB: track 0.00 -> 148.1 mm, vias 0 -> 6
- net SFL: track 0.00 -> 147.1 mm, vias 0 -> 4
- net SLF: track 0.00 -> 144.0 mm, vias 0 -> 4
- net SLB: track 0.00 -> 134.4 mm, vias 0 -> 5
- net SBR: track 0.00 -> 113.4 mm, vias 0 -> 6
- net GND: track 0.00 -> 101.1 mm, vias 0 -> 5
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- added copper zone on layer 1, net +5V
- added copper zone on layer 16, net GND
Other:
- board text added: "???"
- board text added: "Derick Louie"
- board text added: "EB"
- board text added: "EF"
- board text added: "EL"
- board text added: "ER"
- board text added: "Input / Triplet Sheild"
- board text added: "Kevin Kellar"
- board text added: "SBL"
- board text added: "SBR"
- board text added: "SFL"
- board text added: "SFR"
- board text added: "SLF"
- board text added: "SLR"
- board text added: "SRB"
- board text added: "SRF"
- board text added: "TRIG"
