File: hardware/inputsheild_6.brd (EAGLE design)
At the start: 71.1 x 90 mm, 73 parts, among them X1 MKDSN1,5/2-5,08, X2 MKDSN1,5/4-5,08, X3 MKDSN1,5/4-5,08, X4 MKDSN1,5/4-5,08

Commit message: work on sheild 6
Parts:
- added SWITCH_XTRA: MKDSN1,5/2-5,08, con-phoenix-508:MKDSN1,5/2-5,08
- added U$1: NANO, Arduino-clone:NANO
- moved PWM_L1 1.27 mm to (33.0, 16.3)
- flipped COMMON_TERMINAL to the top
- renumbered SFR to VIN, SFR_ to VIN_, SFR__ to VIN__, X1 to SWTICH_LOC, X2 to SWITCH_MAIN, X3 to COMMON_TERMINAL, X4 to ECHO_TERMINAL, _SFR to _VIN
Connections:
- new net VIN: B1.VIN, COMMON_TERMINAL.4, VIN.1, VIN_.1, VIN__.1, _VIN.1
- net +5V: now also COMMON_TERMINAL.2
- net EB: now also ECHO_TERMINAL.3
- net EF: now also ECHO_TERMINAL.1
- net EL: now also ECHO_TERMINAL.2
- net ER: now also ECHO_TERMINAL.4
- net GND: now also COMMON_TERMINAL.1
- net SBL: now also SWITCH_MAIN.3
- net SBR: now also SWTICH_LOC.2
- net SFL: now also SWITCH_MAIN.1
- net SFR: now also SWTICH_LOC.1; no longer VIN.1, VIN_.1, VIN__.1, _VIN.1
- net SLB: now also SWITCH_XTRA.1
- net SLF: now also SWITCH_MAIN.2
- net SRB: now also SWITCH_XTRA.2
- net SRF: now also SWITCH_MAIN.4
- net TRIG: now also COMMON_TERMINAL.3

Commit message: ready to route 6
Parts:
- moved _5V 225.0 mm to (67.3, 4.02), flipped to the bottom, turned to 270 degrees
- moved _VIN 215.6 mm to (67.4, 9.61), flipped to the bottom, turned to 270 degrees
- moved U$1 211.6 mm to (33.0, 62.2), turned to 180 degrees
- moved _SRB 206.3 mm to (67.4, 14.8), flipped to the bottom, turned to 270 degrees
- moved _SRF 197.2 mm to (67.4, 20.1), flipped to the bottom, turned to 270 degrees
- moved _SBL 188.3 mm to (67.3, 25.6), flipped to the bottom, turned to 270 degrees
- moved _SLB 179.9 mm to (67.4, 31.3), flipped to the bottom, turned to 270 degrees
- moved _SLF 171.6 mm to (67.4, 36.1), flipped to the bottom, turned to 270 degrees
- moved _SFL 163.6 mm to (67.4, 41.0), flipped to the bottom, turned to 270 degrees
- moved 5V__ 156.6 mm to (3.66, 4.40), flipped to the bottom, turned to 270 degrees
- moved _A5 156.1 mm to (67.3, 46.4), flipped to the bottom, turned to 270 degrees
- moved _A4 149.2 mm to (67.4, 51.8), flipped to the bottom, turned to 270 degrees
- moved VIN__ 147.3 mm to (3.57, 9.48), flipped to the bottom, turned to 270 degrees
- moved _TRIG 142.7 mm to (67.4, 57.0), flipped to the bottom, turned to 270 degrees
- moved SRB__ 138.4 mm to (3.60, 14.7), flipped to the bottom, turned to 270 degrees
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Connections:
- removed net SLR: B1.D5
- new net +3.3V: B1.3.3V, U$1.3.3V
- new net A3: U$1.A3
- new net AREF: B1.AREF, U$1.AREF
- new net N$11: U$1.A6
- new net N$12: U$1.A7
- new net N$21: U$1.RST1
- new net RST: B1.RES, U$1.RST
- new net RX: B1.RX, U$1.RX1
- new net TX: B1.TX, U$1.TX0
- net +5V: now also U$1.5V
- net A4: now also U$1.A4
- net A5: now also U$1.A5
- net EB: now also U$1.D13
- net EF: now also U$1.D8
- net EL: now also U$1.D12
- net ER: now also U$1.D11
- net GND: now also U$1.GND, U$1.GND1
- net PWM_L: now also U$1.D9
- net PWM_R: now also U$1.D10
- net SBL: now also U$1.D3
- net SBR: now also U$1.A0
- net SFL: now also U$1.D2
- net SFR: now also U$1.A1
- net SLB: now also B1.D5, U$1.D5
- net SLF: now also U$1.D4
- net SRB: now also U$1.A2
- net SRF: now also U$1.D6
- net TRIG: now also U$1.D7
- net VIN: now also U$1.RAW
