File: hardware/inputsheild_6.sch (EAGLE design)
At the start: 73 parts, among them X1 MKDSN1,5/2-5,08, X2 MKDSN1,5/4-5,08, X3 MKDSN1,5/4-5,08, X4 MKDSN1,5/4-5,08

Commit message: work on sheild 6
Parts:
- added SWITCH_XTRA: MKDSN1,5/2-5,08, con-phoenix-508:MKDSN1,5/2-5,08
- added U$1: NANO, Arduino-clone:NANO
- renumbered SFR to VIN, SFR_ to VIN_, SFR__ to VIN__, X1 to SWTICH_LOC, X2 to SWITCH_MAIN, X3 to COMMON_TERMINAL, X4 to ECHO_TERMINAL, _SFR to _VIN
Connections:
- new net VIN: B1.VIN, COMMON_TERMINAL-4.KL, VIN.P, VIN_.P, VIN__.P, _VIN.P
- net +5V: now also COMMON_TERMINAL-2.KL
- net EB: now also ECHO_TERMINAL-3.KL
- net EF: now also ECHO_TERMINAL-1.KL
- net EL: now also ECHO_TERMINAL-2.KL
- net ER: now also ECHO_TERMINAL-4.KL
- net GND: now also COMMON_TERMINAL-1.KL
- net SBL: now also SWITCH_MAIN-3.KL
- net SBR: now also SWTICH_LOC-2.KL
- net SFL: now also SWITCH_MAIN-1.KL
- net SFR: now also SWTICH_LOC-1.KL; no longer VIN.P, VIN_.P, VIN__.P, _VIN.P
- net SLB: now also SWITCH_XTRA-1.KL
- net SLF: now also SWITCH_MAIN-2.KL
- net SRB: now also SWITCH_XTRA-2.KL
- net SRF: now also SWITCH_MAIN-4.KL
- net TRIG: now also COMMON_TERMINAL-3.KL

Commit message: ready to route 6
Connections:
- removed net SLR: B1.*D5
- new net +3.3V: B1.3.3V, U$1.3.3V
- new net A3: U$1.A3
- new net AREF: B1.AREF, U$1.AREF
- new net N$11: U$1.A6
- new net N$12: U$1.A7
- new net N$21: U$1.RST1
- new net RST: B1.RES, U$1.RST
- new net RX: B1.RX, U$1.RX1
- new net TX: B1.TX, U$1.TX0
- net +5V: now also U$1.5.5V
- net A4: now also U$1.A4
- net A5: now also U$1.A5
- net EB: now also U$1.D13
- net EF: now also U$1.D8
- net EL: now also U$1.D12
- net ER: now also U$1.D11
- net GND: now also U$1.GND, U$1.GND2
- net PWM_L: now also U$1.D9
- net PWM_R: now also U$1.D10
- net SBL: now also U$1.D3
- net SBR: now also U$1.A0
- net SFL: now also U$1.D2
- net SFR: now also U$1.A1
- net SLB: now also B1.*D5, U$1.D5
- net SLF: now also U$1.D4
- net SRB: now also U$1.A2
- net SRF: now also U$1.D6
- net TRIG: now also U$1.D7
- net VIN: now also U$1.RAW
