File: hardware/inputsheild_7.brd (EAGLE design)
At the start: 71.1 x 90 mm, 80 parts

Commit message: big reorganize
Parts:
- moved PWM_R1 1.32 mm to (32.9, 13.3)
Routing:
- net +5V: track 0.00 -> 216.3 mm, vias 0 -> 11
- net VIN: track 0.00 -> 173.4 mm, vias 0 -> 4
- net EB: track 0.00 -> 145.8 mm, vias 0 -> 3
- net SLB: track 20.2 -> 165.9 mm, vias 0 -> 3
- net SFL: track 20.2 -> 164.6 mm, vias 0 -> 4
- net SRB: track 0.00 -> 142.7 mm, vias 0 -> 4
- net SLF: track 20.2 -> 157.8 mm, vias 0 -> 4
- net SBL: track 20.2 -> 151.7 mm, vias 0 -> 4
- net SRF: track 20.3 -> 146.6 mm, vias 0 -> 4
- net ER: track 19.6 -> 141.7 mm, vias 0 -> 2
- net EL: track 19.6 -> 139.6 mm, vias 0 -> 3
- net A5: track 0.00 -> 118.0 mm, vias 0 -> 3
- net EF: track 19.6 -> 134.2 mm, vias 0 -> 2
- net PWM_R: track 19.6 -> 131.5 mm, vias 0 -> 1
- net A4: track 0.00 -> 102.2 mm, vias 0 -> 4
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Other:
- board text added: "+5v"
- board text added: "??"
